File: Entrenadora Digital/ed_esquema.sch (EAGLE design)
At the start: 0 parts

Commit message: Entrenadora Digital con Arduino
Parts:
- added B1: ARDUINO_NANO, treser_lib:ARDUINO_NANO
- added IC1: DHT11, treser_lib:DHT11
- added LED1: (no value), treser_lib:LED3MM
- added M1: SERVO, treser_lib:SERVO
- added R1: (no value), treser_lib:RESISTOR-EU0204/7
- added R2: (no value), pot:TRIM_EU-B64W
- added S1: (no value), treser_lib:SWITCH
Changed lines of the file:
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@@
 <schematic xreflabel="%F%N/%S.%C%R" xrefpart="/%S.%C%R">
 <attributes>
+<attribute name="CDESIGNER" value="Apellido, Nombre"/>
+<attribute name="CNAME" value="ENTRENADORA DIGITAL"/>
+<attribute name="CREVISION" value="1.0"/>
+<attribute name="CSCHO" value="ESCUELA"/>
 </attributes>
 <variantdefs>
@@
 <parts>
 <part name="FRAME1" library="treser_lib" deviceset="FRAME-A4L" device=""/>
+<part name="B1" library="treser_lib" deviceset="ARDUINO_NANO" device=""/>
+<part name="LED1" library="treser_lib" deviceset="LED" device="3MM"/>
+<part name="M1" library="treser_lib" deviceset="SERVO" device=""/>
+<part name="R1" library="treser_lib" deviceset="RESISTOR-EU" device="0204/7"/>
+<part name="IC1" library="treser_lib" deviceset="DHT11" device=""/>
+<part name="R2" library="pot" deviceset="TRIM_EU-" device="B64W"/>
+<part name="S1" library="treser_lib" deviceset="SWITCH" device=""/>
+<part name="SUPPLY1" library="supply2" deviceset="GND" device=""/>
+<part name="P+1" library="supply1" deviceset="VCC" device=""/>
 </parts>
 <sheets>
@@
 <instances>
 <instance part="FRAME1" gate="G$1" x="2.54" y="2.54"/>
+<instance part="B1" gate="G$1" x="142.24" y="99.06"/>
+<instance part="LED1" gate="G$1" x="101.6" y="116.84"/>
+<instance part="M1" gate="G$1" x="203.2" y="83.82"/>
+<instance part="R1" gate="G$1" x="96.52" y="104.14"/>
+<instance part="IC1" gate="G$1" x="193.04" y="119.38"/>
+<instance part="R2" gate="1" x="111.76" y="76.2"/>
+<instance part="S1" gate="1" x="81.28" y="83.82"/>
+<instance part="SUPPLY1" gate="GND" x="104.14" y="50.8"/>
+<instance part="P+1" gate="VCC" x="101.6" y="60.96"/>
 </instances>
 <busses>

Commit message: Entrenadora Digital
Parts:
- removed M1: SERVO, treser_lib:SERVO
- added IC2: (no value), uln-udn:ULN2803A
- added JP1: I2C, pinhead:PINHD-1X4
- added JP2: SPI, pinhead:PINHD-1X6
- added LED2, LED3, LED4, LED5, LED6, LED7, LED8: (no value), treser_lib:LED3MM
- added R10, R4, R5, R6, R7, R8, R9: (no value), treser_lib:RESISTOR-EU0204/7
- added R3: (no value), pot:TRIM_EU-B64W
- added S2, S3, S4: (no value), treser_lib:SWITCH
Connections:
- new net N$1: JP1.1
- new net N$10: JP2.6
- new net N$11: LED8.A, R10.2
- new net N$2: JP1.2
- new net N$3: JP1.3
- new net N$4: JP1.4
- new net N$5: JP2.1
- new net N$6: JP2.2
- new net N$7: JP2.3
- new net N$8: JP2.4
- new net N$9: JP2.5
Other:
- moved on the sheet: IC1, LED1, R1, S1
Changed lines of the file:
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@@
 <part name="B1" library="treser_lib" deviceset="ARDUINO_NANO" device=""/>
 <part name="LED1" library="treser_lib" deviceset="LED" device="3MM"/>
-<part name="M1" library="treser_lib" deviceset="SERVO" device=""/>
 <part name="R1" library="treser_lib" deviceset="RESISTOR-EU" device="0204/7"/>
 <part name="IC1" library="treser_lib" deviceset="DHT11" device=""/>
@@
 <part name="SUPPLY1" library="supply2" deviceset="GND" device=""/>
 <part name="P+1" library="supply1" deviceset="VCC" device=""/>
+<part name="IC2" library="uln-udn" deviceset="ULN2803A" device=""/>
+<part name="S2" library="treser_lib" deviceset="SWITCH" device=""/>
+<part name="S3" library="treser_lib" deviceset="SWITCH" device=""/>
+<part name="S4" library="treser_lib" deviceset="SWITCH" device=""/>
+<part name="R3" library="pot" deviceset="TRIM_EU-" device="B64W"/>
+<part name="JP1" library="pinhead" deviceset="PINHD-1X4" device="" value="I2C"/>
+<part name="JP2" library="pinhead" deviceset="PINHD-1X6" device="" value="SPI"/>
+<part name="LED2" library="treser_lib" deviceset="LED" device="3MM"/>
+<part name="LED3" library="treser_lib" deviceset="LED" device="3MM"/>
+<part name="LED4" library="treser_lib" deviceset="LED" device="3MM"/>
+<part name="R4" library="treser_lib" deviceset="RESISTOR-EU" device="0204/7"/>
+<part name="R5" library="treser_lib" deviceset="RESISTOR-EU" device="0204/7"/>
+<part name="R6" library="treser_lib" deviceset="RESISTOR-EU" device="0204/7"/>
+<part name="R7" library="treser_lib" deviceset="RESISTOR-EU" device="0204/7"/>
+<part name="R8" library="treser_lib" deviceset="RESISTOR-EU" device="0204/7"/>
+<part name="R9" library="treser_lib" deviceset="RESISTOR-EU" device="0204/7"/>
+<part name="LED5" library="treser_lib" deviceset="LED" device="3MM"/>
+<part name="LED6" library="treser_lib" deviceset="LED" device="3MM"/>
+<part name="LED7" library="treser_lib" deviceset="LED" device="3MM"/>
+<part name="LED8" library="treser_lib" deviceset="LED" device="3MM"/>
+<part name="R10" library="treser_lib" deviceset="RESISTOR-EU" device="0204/7"/>
 </parts>
 <sheets>
@@
 <instance part="FRAME1" gate="G$1" x="2.54" y="2.54"/>
 <instance part="B1" gate="G$1" x="142.24" y="99.06"/>
-<instance part="LED1" gate="G$1" x="101.6" y="116.84"/>
-<instance part="M1" gate="G$1" x="203.2" y="83.82"/>
-<instance part="R1" gate="G$1" x="96.52" y="104.14"/>
-<instance part="IC1" gate="G$1" x="193.04" y="119.38"/>
+<instance part="LED1" gate="G$1" x="93.98" y="147.32" rot="R90"/>
+<instance part="R1" gate="G$1" x="83.82" y="147.32"/>
+<instance part="IC1" gate="G$1" x="228.6" y="116.84"/>
 <instance part="R2" gate="1" x="111.76" y="76.2"/>
-<instance part="S1" gate="1" x="81.28" y="83.82"/>
+<instance part="S1" gate="1" x="43.18" y="106.68"/>
 <instance part="SUPPLY1" gate="GND" x="104.14" y="50.8"/>
 <instance part="P+1" gate="VCC" x="101.6" y="60.96"/>
+<instance part="IC2" gate="G$1" x="177.8" y="101.6"/>
+<instance part="S2" gate="1" x="43.18" y="93.98"/>
+<instance part="S3" gate="1" x="43.18" y="78.74"/>
+<instance part="S4" gate="1" x="43.18" y="66.04"/>
+<instance part="R3" gate="1" x="119.38" y="66.04"/>
+<instance part="JP1" gate="A" x="228.6" y="78.74"/>
+<instance part="JP2" gate="A" x="228.6" y="55.88"/>
+<instance part="LED2" gate="G$1" x="93.98" y="139.7" rot="R90"/>
+<instance part="LED3" gate="G$1" x="93.98" y="132.08" rot="R90"/>
+<instance part="LED4" gate="G$1" x="93.98" y="124.46" rot="R90"/>
+<instance part="R4" gate="G$1" x="83.82" y="139.7"/>
+<instance part="R5" gate="G$1" x="83.82" y="132.08"/>
+<instance part="R6" gate="G$1" x="83.82" y="124.46"/>
+<instance part="R7" gate="G$1" x="83.82" y="116.84"/>
+<instance part="R8" gate="G$1" x="83.82" y="109.22"/>
+<instance part="R9" gate="G$1" x="83.82" y="101.6"/>
+<instance part="LED5" gate="G$1" x="93.98" y="116.84" rot="R90"/>
+<instance part="LED6" gate="G$1" x="93.98" y="109.22" rot="R90"/>
+<instance part="LED7" gate="G$1" x="93.98" y="101.6" rot="R90"/>
+<instance part="LED8" gate="G$1" x="93.98" y="93.98" rot="R90"/>
+<instance part="R10" gate="G$1" x="83.82" y="93.98"/>
 </instances>
 <busses>
 </busses>
 <nets>
+<net name="N$1" class="0">
+<segment>
+<pinref part="JP1" gate="A" pin="1"/>
+<wire x1="226.06" y1="83.82" x2="213.36" y2="83.82" width="0.1524" layer="91"/>
+</segment>
+</net>
+<net name="N$2" class="0">
+<segment>
+<pinref part="JP1" gate="A" pin="2"/>
+<wire x1="226.06" y1="81.28" x2="213.36" y2="81.28" width="0.1524" layer="91"/>
+</segment>
+</net>
+<net name="N$3" class="0">
+<segment>
+<pinref part="JP1" gate="A" pin="3"/>
+<wire x1="226.06" y1="78.74" x2="213.36" y2="78.74" width="0.1524" layer="91"/>
+</segment>
+</net>
+<net name="N$4" class="0">
+<segment>
+<pinref part="JP1" gate="A" pin="4"/>
+<wire x1="226.06" y1="76.2" x2="213.36" y2="76.2" width="0.1524" layer="91"/>
+</segment>
+</net>
+<net name="N$5" class="0">
+<segment>
+<pinref part="JP2" gate="A" pin="1"/>
+<wire x1="226.06" y1="63.5" x2="213.36" y2="63.5" width="0.1524" layer="91"/>
+</segment>
+</net>
+<net name="N$6" class="0">
+<segment>
+<pinref part="JP2" gate="A" pin="2"/>
+<wire x1="226.06" y1="60.96" x2="213.36" y2="60.96" width="0.1524" layer="91"/>
+</segment>
+</net>
+<net name="N$7" class="0">
+<segment>
+<pinref part="JP2" gate="A" pin="3"/>
+<wire x1="226.06" y1="58.42" x2="213.36" y2="58.42" width="0.1524" layer="91"/>
+</segment>
+</net>
+<net name="N$8" class="0">
+<segment>
+<pinref part="JP2" gate="A" pin="4"/>
+<wire x1="226.06" y1="55.88" x2="213.36" y2="55.88" width="0.1524" layer="91"/>
+</segment>
+</net>
+<net name="N$9" class="0">
+<segment>
+<pinref part="JP2" gate="A" pin="5"/>
+<wire x1="226.06" y1="53.34" x2="213.36" y2="53.34" width="0.1524" layer="91"/>
+</segment>
+</net>
+<net name="N$10" class="0">
+<segment>
+<pinref part="JP2" gate="A" pin="6"/>
+<wire x1="226.06" y1="50.8" x2="213.36" y2="50.8" width="0.1524" layer="91"/>
+</segment>
+</net>
+<net name="N$11" class="0">
+<segment>
+<pinref part="LED8" gate="G$1" pin="A"/>
+<pinref part="R10" gate="G$1" pin="2"/>
+<wire x1="88.9" y1="93.98" x2="91.44" y2="93.98" width="0.1524" layer="91"/>
+</segment>
+</net>
 </nets>
 </sheet>

Commit message: Diagrama esquemático
Parts:
- removed IC1: DHT11, treser_lib:DHT11
- added JP3: VIN, jumper:JP1E
- added R11, R12, R13, R14: 10k, treser_lib:RESISTOR-EU0204/7
- added X1, X2, X3, X4, X5: (no value), treser_lib:BORNERA_AK500/2
- B1: value ARDUINO_NANO -> ARDUINO NANO
- IC2: value (none) -> ULN2803
- R1, R10, R4, R5, R6, R7, R8, R9: value (none) -> 330
- R2, R3: value (none) -> 10k
Connections:
- removed net N$10: JP2.6
- removed net N$2: JP1.2
- removed net N$4: JP1.4
- removed net N$6: JP2.2
- removed net N$8: JP2.4
- removed net N$9: JP2.5
- new net A0: B1.A0, S4.S1
- new net A1: B1.A1, S3.S1
- new net A2: B1.A2, S2.S1
- new net A3: B1.A3, S1.S1
- new net A6: B1.A6, R2.S
- new net A7: B1.A7, R3.S
- new net D2: B1.D2, IC2.I1, R1.1
- new net D3: B1.D3, IC2.I2, R4.1
- new net D4: B1.D4, IC2.I3, R5.1
- new net D5: B1.D5, IC2.I4, R6.1
- new net D6: B1.D6, IC2.I5, R7.1
- new net D7: B1.D7, IC2.I6, R8.1
- new net D8: B1.D8, IC2.I7, R9.1
- new net D9: B1.D9, IC2.I8, R10.1
- new net GND: B1.GND, IC2.GND, JP1.4, JP2.6, LED1.C, LED2.C, LED3.C, LED4.C, LED5.C, LED6.C, LED7.C, LED8.C, R2.A, R3.A, S1.P, S1.P1, S2.P, S2.P1, S3.P, S3.P1, S4.P, S4.P1, X5-2.KL
- new net MISO: B1.D12, JP2.3
- new net MOSI: B1.D11, JP2.4
- new net N$12: LED1.A, R1.2
- new net N$13: LED2.A, R4.2
- new net N$14: LED3.A, R5.2
- new net N$15: LED4.A, R6.2
- new net N$16: LED5.A, R7.2
- new net N$17: LED6.A, R8.2
- new net N$18: LED7.A, R9.2
- new net N$24: IC2.O1, X1-1.KL
- new net N$25: IC2.O2, X1-2.KL
- new net N$26: IC2.O3, X2-1.KL
- new net N$27: IC2.O4, X2-2.KL
- new net N$28: IC2.O5, X3-1.KL
- new net N$29: IC2.O6, X3-2.KL
- new net N$30: IC2.O7, X4-1.KL
- new net N$31: IC2.O8, X4-2.KL
- new net N$32: IC2.CD+, JP3.1, X5-1.KL
- new net SCK: B1.D13, JP2.2
- new net SCL: B1.A5/SCL, JP1.2
- new net SDA: B1.A4/SDA, JP1.3
- new net SS: B1.D10, JP2.5
- new net VCC: B1.5V, JP1.1, JP2.1, R11.2, R12.2, R13.2, R14.2, R2.E, R3.E
- new net VIN: B1.VIN, JP3.2
- net N$1: now also R11.1, S1.S; no longer JP1.1
- net N$3: now also R12.1, S2.S; no longer JP1.3
- net N$5: now also R14.1, S3.S; no longer JP2.1
- net N$7: now also R13.1, S4.S; no longer JP2.3
Other:
- moved on the sheet: B1, IC2, JP1, JP2, LED1, LED2, LED3, LED4, LED5, LED6, LED7, LED8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
