File: Robotec/MUBI-BOT/mubi-ESP32-36.sch (EAGLE design)
At the start: 37 parts, among them IC1 L293D, IC2 7805T

Commit message: update mubi-bot
Parts:
- removed PAD11, PAD12, PAD13, PAD14: WIREPAD1,6/0,8, wirepad:WIREPAD1,6/0,8
- added R3, R4: 1, resistor:R-EU_0207/10
Connections:
- removed net GPIO16/RX2: J4.1, X4-1.KL
- removed net GPIO17/TX2: J2.9, X2-4.KL
- new net GPIO18: J2.7, X4-1.KL
- new net GPIO19: J2.6, X2-4.KL
- new net N$1: J4.2, R3.2
- new net N$2: J4.1, R4.2
- net CM11: now also R4.1; no longer J2.6, PAD13.P, PAD14.P
- net CM12: now also J2.9; no longer J4.2
- net ENAM1: now also R3.1; no longer J2.7, PAD11.P, PAD12.P
Other:
- moved on the sheet: MPU6050
Changed lines of the file:
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@@
 <part name="R1" library="rcl" deviceset="R-EU_" device="0207/7" value="4K7"/>
 <part name="R2" library="rcl" deviceset="R-EU_" device="0207/7" value="4K7"/>
+<part name="R3" library="resistor" deviceset="R-EU_" device="0207/10" value="1"/>
+<part name="R4" library="resistor" deviceset="R-EU_" device="0207/10" value="1"/>
 <part name="C1" library="resistor" deviceset="CPOL-EU" device="E2.5-6"/>
 <part name="C2" library="rcl" deviceset="C-EU" device="025-025X050"/>
@@
 <part name="PAD9" library="wirepad" deviceset="WIREPAD" device="1,6/0,8" value="WIREPAD1,6/0,8"/>
 <part name="PAD10" library="wirepad" deviceset="WIREPAD" device="1,6/0,8" value="WIREPAD1,6/0,8"/>
-<part name="PAD11" library="wirepad" deviceset="WIREPAD" device="1,6/0,8" value="WIREPAD1,6/0,8"/>
-<part name="PAD12" library="wirepad" deviceset="WIREPAD" device="1,6/0,8" value="WIREPAD1,6/0,8"/>
-<part name="PAD13" library="wirepad" deviceset="WIREPAD" device="1,6/0,8" value="WIREPAD1,6/0,8"/>
-<part name="PAD14" library="wirepad" deviceset="WIREPAD" device="1,6/0,8" value="WIREPAD1,6/0,8"/>
 </parts>
 <sheets>
@@
 <attribute name="VALUE" x="69.215" y="63.627" size="1.778" layer="96" rot="R180"/>
 </instance>
+<instance part="R3" gate="G$1" x="66.675" y="40.005" smashed="yes">
+<attribute name="NAME" x="61.595" y="37.0586" size="1.778" layer="95"/>
+<attribute name="VALUE" x="66.675" y="39.243" size="1.778" layer="96"/>
+</instance>
+<instance part="R4" gate="G$1" x="66.675" y="42.545" smashed="yes">
+<attribute name="NAME" x="61.595" y="43.4086" size="1.778" layer="95"/>
+<attribute name="VALUE" x="66.675" y="41.783" size="1.778" layer="96"/>
+</instance>
 <instance part="C1" gate="G$1" x="62.865" y="109.22"/>
 <instance part="C2" gate="G$1" x="32.385" y="109.22"/>
@@
 <attribute name="VALUE" x="203.708" y="118.872" size="1.778" layer="96" rot="R180"/>
 </instance>
-<instance part="MPU6050" gate="G$1" x="170.815" y="43.18"/>
+<instance part="MPU6050" gate="G$1" x="55.88" y="88.9"/>
 <instance part="R5" gate="G$1" x="104.775" y="92.71" smashed="yes">
 <attribute name="NAME" x="98.425" y="93.5736" size="1.778" layer="95"/>
@@
 <attribute name="NAME" x="191.008" y="95.9358" size="1.778" layer="95" rot="R180"/>
 <attribute name="VALUE" x="203.073" y="93.472" size="1.778" layer="96" rot="R180"/>
-</instance>
-<instance part="PAD11" gate="G$1" x="10.795" y="83.82" smashed="yes">
-<attribute name="NAME" x="0.762" y="82.4992" size="1.778" layer="95"/>
-<attribute name="VALUE" x="0.762" y="79.248" size="1.778" layer="96"/>
-</instance>
-<instance part="PAD12" gate="G$1" x="40.005" y="83.82" smashed="yes" rot="R180">
-<attribute name="NAME" x="50.673" y="85.1408" size="1.778" layer="95" rot="R180"/>
-<attribute name="VALUE" x="58.293" y="81.407" size="1.778" layer="96" rot="R180"/>
-</instance>
-<instance part="PAD13" gate="G$1" x="11.43" y="92.71" smashed="yes">
-<attribute name="NAME" x="1.397" y="91.3892" size="1.778" layer="95"/>
-<attribute name="VALUE" x="1.397" y="88.773" size="1.778" layer="96"/>
-</instance>
-<instance part="PAD14" gate="G$1" x="40.005" y="92.71" smashed="yes" rot="R180">
-<attribute name="NAME" x="50.673" y="94.0308" size="1.778" layer="95" rot="R180"/>
-<attribute name="VALUE" x="58.293" y="90.297" size="1.778" layer="96" rot="R180"/>
 </instance>
 </instances>
@@
 <segment>
 <pinref part="MPU6050" gate="G$1" pin="2"/>
-<wire x1="178.435" y1="40.64" x2="179.705" y2="40.64" width="0.1524" layer="91"/>
-<label x="179.705" y="40.64" size="1.778" layer="95" xref="yes"/>
+<wire x1="63.5" y1="86.36" x2="64.77" y2="86.36" width="0.1524" layer="91"/>
+<label x="64.77" y="86.36" size="1.778" layer="95" xref="yes"/>
 </segment>
 <segment>
@@
 <segment>
 <pinref part="MPU6050" gate="G$1" pin="1"/>
-<wire x1="178.435" y1="38.1" x2="179.705" y2="38.1" width="0.1524" layer="91"/>
-<label x="179.705" y="38.1" size="1.778" layer="95" xref="yes"/>
+<wire x1="63.5" y1="83.82" x2="64.77" y2="83.82" width="0.1524" layer="91"/>
+<label x="64.77" y="83.82" size="1.778" layer="95" xref="yes"/>
 </segment>
 </net>
@@
 </segment>
 <segment>
-<pinref part="J4" gate="G$1" pin="2"/>
-<wire x1="73.025" y1="40.005" x2="71.755" y2="40.005" width="0.1524" layer="91"/>
-<label x="71.755" y="40.005" size="1.778" layer="95" rot="R180" xref="yes"/>
+<pinref part="J2" gate="G$2" pin="9"/>
+<wire x1="73.025" y1="48.26" x2="71.755" y2="48.26" width="0.1524" layer="91"/>
+<label x="71.755" y="48.26" size="1.778" layer="95" rot="R180" xref="yes"/>
 </segment>
 </net>
@@
 </segment>
 <segment>
-<pinref part="J2" gate="G$2" pin="6"/>
-<wire x1="73.025" y1="55.88" x2="71.755" y2="55.88" width="0.1524" layer="91"/>
-<label x="71.755" y="55.88" size="1.778" layer="95" rot="R180" xref="yes"/>
-</segment>
-<segment>
-<pinref part="PAD13" gate="G$1" pin="P"/>
-<pinref part="PAD14" gate="G$1" pin="P"/>
-<wire x1="13.97" y1="92.71" x2="20.955" y2="92.71" width="0.1524" layer="91"/>
-<wire x1="20.955" y1="92.71" x2="37.465" y2="92.71" width="0.1524" layer="91"/>
-<wire x1="20.955" y1="92.71" x2="20.955" y2="95.25" width="0.1524" layer="91"/>
-<wire x1="20.955" y1="95.25" x2="23.495" y2="95.25" width="0.1524" layer="91"/>
-<label x="23.495" y="95.25" size="1.778" layer="95" xref="yes"/>
+<pinref part="R4" gate="G$1" pin="1"/>
+<wire x1="61.595" y1="42.545" x2="60.325" y2="42.545" width="0.1524" layer="91"/>
+<label x="60.325" y="42.545" size="1.778" layer="95" rot="R180" xref="yes"/>
 </segment>
 </net>
@@
 </segment>
 <segment>
-<pinref part="J2" gate="G$2" pin="7"/>
-<wire x1="73.025" y1="53.34" x2="71.755" y2="53.34" width="0.1524" layer="91"/>
-<label x="71.755" y="53.34" size="1.778" layer="95" rot="R180" xref="yes"/>
-</segment>
-<segment>
-<pinref part="PAD12" gate="G$1" pin="P"/>
-<pinref part="PAD11" gate="G$1" pin="P"/>
-<wire x1="37.465" y1="83.82" x2="20.955" y2="83.82" width="0.1524" layer="91"/>
-<wire x1="20.955" y1="83.82" x2="13.335" y2="83.82" width="0.1524" layer="91"/>
-<wire x1="20.955" y1="83.82" x2="20.955" y2="86.36" width="0.1524" layer="91"/>
-<wire x1="20.955" y1="86.36" x2="23.495" y2="86.36" width="0.1524" layer="91"/>
-<label x="24.13" y="86.36" size="1.778" layer="95" xref="yes"/>
+<pinref part="R3" gate="G$1" pin="1"/>
+<wire x1="61.595" y1="40.005" x2="60.325" y2="40.005" width="0.1524" layer="91"/>
+<label x="60.325" y="40.005" size="1.778" layer="95" rot="R180" xref="yes"/>
+</segment>
+</net>
+<net name="N$1" class="0">
+<segment>
+<pinref part="J4" gate="G$1" pin="2"/>
+<wire x1="73.025" y1="40.005" x2="71.755" y2="40.005" width="0.1524" layer="91"/>
+<pinref part="R3" gate="G$1" pin="2"/>
+</segment>
+</net>
+<net name="N$2" class="0">
+<segment>
+<pinref part="J4" gate="G$1" pin="1"/>
+<wire x1="73.025" y1="42.545" x2="71.755" y2="42.545" width="0.1524" layer="91"/>
+<pinref part="R4" gate="G$1" pin="2"/>
 </segment>
 </net>
@@
 <segment>
 <pinref part="MPU6050" gate="G$1" pin="3"/>
-<wire x1="178.435" y1="43.18" x2="179.705" y2="43.18" width="0.1524" layer="91"/>
-<label x="179.705" y="43.18" size="1.778" layer="95" xref="yes"/>
+<wire x1="63.5" y1="88.9" x2="64.77" y2="88.9" width="0.1524" layer="91"/>
+<label x="64.77" y="88.9" size="1.778" layer="95" xref="yes"/>
 </segment>
 <segment>
@@
 <segment>
 <pinref part="MPU6050" gate="G$1" pin="4"/>
-<wire x1="178.435" y1="45.72" x2="179.705" y2="45.72" width="0.1524" layer="91"/>
-<label x="179.705" y="45.72" size="1.778" layer="95" xref="yes"/>
+<wire x1="63.5" y1="91.44" x2="64.77" y2="91.44" width="0.1524" layer="91"/>
+<label x="64.77" y="91.44" size="1.778" layer="95" xref="yes"/>
 </segment>
 <segment>
@@
 </segment>
 </net>
+<net name="GPIO19" class="0">
+<segment>
+<pinref part="J2" gate="G$2" pin="6"/>
+<wire x1="73.025" y1="55.88" x2="71.12" y2="55.88" width="0.1524" layer="91"/>
+<label x="71.12" y="55.88" size="1.778" layer="95" rot="R180" xref="yes"/>
+</segment>
+<segment>
+<pinref part="X2" gate="-4" pin="KL"/>
+<wire x1="172.72" y1="110.49" x2="173.99" y2="110.49" width="0.1524" layer="91"/>
+<label x="173.99" y="110.49" size="1.778" layer="95" xref="yes"/>
+</segment>
+</net>
+<net name="GPIO18" class="0">
+<segment>
+<pinref part="J2" gate="G$2" pin="7"/>
+<wire x1="73.025" y1="53.34" x2="71.12" y2="53.34" width="0.1524" layer="91"/>
+<label x="71.12" y="53.34" size="1.778" layer="95" rot="R180" xref="yes"/>
+</segment>
+<segment>
+<pinref part="X4" gate="-1" pin="KL"/>
+<wire x1="172.72" y1="105.41" x2="173.99" y2="105.41" width="0.1524" layer="91"/>
+<label x="173.99" y="105.41" size="1.778" layer="95" xref="yes"/>
+</segment>
+</net>
 <net name="N$3" class="0">
 <segment>
@@
 </segment>
 </net>
-<net name="GPIO17/TX2" class="0">
-<segment>
-<pinref part="J2" gate="G$2" pin="9"/>
-<wire x1="73.025" y1="48.26" x2="71.12" y2="48.26" width="0.1524" layer="91"/>
-<label x="71.755" y="48.26" size="1.778" layer="95" rot="R180" xref="yes"/>
-</segment>
-<segment>
-<pinref part="X2" gate="-4" pin="KL"/>
-<wire x1="172.72" y1="110.49" x2="173.99" y2="110.49" width="0.1524" layer="91"/>
-<label x="173.99" y="110.49" size="1.778" layer="95" xref="yes"/>
-</segment>
-</net>
-<net name="GPIO16/RX2" class="0">
-<segment>
-<pinref part="J4" gate="G$1" pin="1"/>
-<wire x1="73.025" y1="42.545" x2="71.755" y2="42.545" width="0.1524" layer="91"/>
-<label x="71.755" y="42.545" size="1.778" layer="95" rot="R180" xref="yes"/>
-</segment>
-<segment>
-<pinref part="X4" gate="-1" pin="KL"/>
-<wire x1="172.72" y1="105.41" x2="174.625" y2="105.41" width="0.1524" layer="91"/>
-<label x="174.625" y="105.41" size="1.778" layer="95" xref="yes"/>
-</segment>
-</net>
