File: Robotec/MUBI-BOT/mubi-bot-PICO-3.sch (EAGLE design)
At the start: 20 parts, among them IC1 L293E, IC2 7805T

Commit message: update MUBI-BOT
Other:
- note removed: "PLACA ROBOT RASPBERRY PICO"
Changed lines of the file:
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@@
 <setting verticaltext="up"/>
 </settings>
-<grid distance="0.1" unitdist="inch" unit="inch" style="lines" multiple="1" display="no" altdistance="0.01" altunitdist="inch" altunit="inch"/>
+<grid distance="25" unitdist="mil" unit="mil" style="lines" multiple="1" display="yes" altdistance="0.01" altunitdist="inch" altunit="inch"/>
 <layers>
 <layer number="1" name="Top" color="4" fill="1" visible="no" active="no"/>
@@
 <sheet>
 <plain>
-<text x="60.96" y="129.54" size="2.54" layer="91">PLACA ROBOT RASPBERRY PICO</text>
 </plain>
 <instances>
