File: Robotec/MUBI-BOT/mubi-ESP32-38.sch (EAGLE design)
At the start: 20 parts, among them IC1 L293D, IC2 7805T

Commit message: update MUBI-BOT
Parts:
- added J5, J6: (no value), con-amp:MTA02-100
- added PAD5, PAD6, PAD7, PAD8: WIREPAD1,6/0,9, wirepad:WIREPAD1,6/0,9
- J3, J4: device con-amp:MTA10-100 -> con-amp:MTA05-100
- PAD1, PAD2, PAD3, PAD4: value WIREPAD2,15/1,0 -> WIREPAD1,6/0,9; device wirepad:WIREPAD2,15/1,0 -> wirepad:WIREPAD1,6/0,9
Connections:
- removed net N$1: PAD1.P, PAD2.P
- removed net N$2: PAD3.P, PAD4.P
- new net +3.3V: J1.1
- new net +5V: C1.+, IC1.VCC1, IC2.VO, J5.2, PAD1.P, PAD2.P, X3-1.KL
- new net +VBAT: IC1.VCC2
- new net CM11: IC1.1A, J2.1, PAD7.P, PAD8.P
- new net CM12: IC1.2A, J2.2
- new net CM21: IC1.4A, J3.3, PAD3.P, PAD4.P
- new net CM22: IC1.3A, J3.2
- new net ENAM1: IC1.1-2EN, J4.4, PAD5.P, PAD6.P
- new net ENAM2: IC1.3-4EN, J3.1
- new net GND: C1.-, C2.2, IC1.GND1, IC1.GND2, IC1.GND3, IC1.GND4, IC2.GND, J2.3, J2.9, J3.5, X3-2.KL
- new net GPIO23: J2.8
- new net M11: IC1.1Y, X4-4.KL
- new net M12: IC1.2Y, X4-3.KL
- new net M21: IC1.4Y, X3-3.KL
- new net M22: IC1.3Y, X3-4.KL
- new net N$3: C2.1, IC2.VI
- new net SCL: J2.7
- new net SDA: J2.4
Other:
- note added: "3.ADC1-0/GPI36"
- note added: "4.ADC1-3/GPI39"
- note added: "5.GPI34"
- note added: "6.GPI35"
- note added: "PLACA ROBOT CON ESP32_38 PINES"
- note removed: "3.ADC1-0/GPIO36"
- note removed: "4.ADC1-3/GPIO39"
- note removed: "5.GPIO34"
- note removed: "6.GPIO35"
- moved on the sheet: C1, C2, IC1, PAD1, PAD2, PAD3, PAD4, R1, R2, R3, R4, X1-1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

Commit message: update MUBI-BOT
Parts:
- added J7: (no value), con-amp:MTA04-100
- added PAD10, PAD11, PAD12, PAD9: WIREPAD1,6/0,9, wirepad:WIREPAD1,6/0,9
- added R5, R6: (no value), resistor:R-EU_0204/5
- added R7, R8: (no value), resistor:R-EU_0207/7
- R1, R2, R3, R4: device resistor:R-EU_0207/10 -> resistor:R-EU_0204/5
Connections:
- removed net GPIO23: J2.8
- new net AUX2: J1.9, X3-5.KL
- new net N$1: R1.1, X1-3.KL
- new net N$2: R3.1, X1-2.KL
- new net N$4: J1.3, X1-4.KL
- new net USON1: J1.4, R1.2, R2.2
- new net USON2: J1.5, R3.2, R4.2
- new net USON3: J1.6, R5.2, R6.2
- net +3.3V: now also J7.1, R7.2, R8.2, X2-1.KL
- net +VBAT: now also C2.1, IC2.VI, PAD10.P, PAD11.P, PAD12.P, PAD9.P, X4-6.KL
- net CM11: now also J2.2; no longer J2.1
- net CM12: now also J2.1; no longer J2.2
- net CM22: now also J3.1; no longer J3.2
- net ENAM2: now also J3.2; no longer J3.1
- net GND: now also J7.2, R2.1, R4.1, R6.1, X2-2.KL, X3-6.KL, X4-5.KL
- net N$3: now also R5.1, X1-1.KL; no longer C2.1, IC2.VI
- net SCL: now also J7.3, R7.1, X2-3.KL
- net SDA: now also J7.4, R8.1, X2-4.KL
Other:
- note added: "13.GPIO12"
- moved on the sheet: C1, C2, IC2, R1, R2, R3, R4, X1-1, X1-2, X1-3, X1-4, X3-1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

Commit message: update sch & brd
Parts:
- C1: value (none) -> 10uF/16V
- C2: value (none) -> 100nF
- R1, R3, R5: value (none) -> 5K6
- R2, R4, R6: value (none) -> 10K
- R7, R8: value (none) -> 4K7
Connections:
- net AUX2 renamed AUX3
- new net AUX1/TX2: J4.4, X4-1.KL
- new net AUX2/RX2: J4.3, X4-2.KL
- net ENAM1: now also J4.2; no longer J4.4
Changed lines of the file:
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@@
 <part name="PAD3" library="wirepad" deviceset="WIREPAD" device="1,6/0,9" value="WIREPAD1,6/0,9"/>
 <part name="PAD4" library="wirepad" deviceset="WIREPAD" device="1,6/0,9" value="WIREPAD1,6/0,9"/>
-<part name="C1" library="resistor" deviceset="CPOL-EU" device="E2.5-6"/>
-<part name="C2" library="rcl" deviceset="C-EU" device="025-025X050"/>
+<part name="C1" library="resistor" deviceset="CPOL-EU" device="E2.5-6" value="10uF/16V"/>
+<part name="C2" library="rcl" deviceset="C-EU" device="025-025X050" value="100nF"/>
 <part name="X1" library="con-ptr500" deviceset="AK500/4-H" device=""/>
 <part name="X2" library="con-ptr500" deviceset="AK500/4-H" device=""/>
@@
 <part name="PAD7" library="wirepad" deviceset="WIREPAD" device="1,6/0,9" value="WIREPAD1,6/0,9"/>
 <part name="PAD8" library="wirepad" deviceset="WIREPAD" device="1,6/0,9" value="WIREPAD1,6/0,9"/>
-<part name="R1" library="resistor" deviceset="R-EU_" device="0204/5"/>
-<part name="R2" library="resistor" deviceset="R-EU_" device="0204/5"/>
-<part name="R3" library="resistor" deviceset="R-EU_" device="0204/5"/>
-<part name="R4" library="resistor" deviceset="R-EU_" device="0204/5"/>
-<part name="R5" library="resistor" deviceset="R-EU_" device="0204/5"/>
-<part name="R6" library="resistor" deviceset="R-EU_" device="0204/5"/>
+<part name="R1" library="resistor" deviceset="R-EU_" device="0204/5" value="5K6"/>
+<part name="R2" library="resistor" deviceset="R-EU_" device="0204/5" value="10K"/>
+<part name="R3" library="resistor" deviceset="R-EU_" device="0204/5" value="5K6"/>
+<part name="R4" library="resistor" deviceset="R-EU_" device="0204/5" value="10K"/>
+<part name="R5" library="resistor" deviceset="R-EU_" device="0204/5" value="5K6"/>
+<part name="R6" library="resistor" deviceset="R-EU_" device="0204/5" value="10K"/>
 <part name="GND7" library="supply1" deviceset="GND" device=""/>
 <part name="GND8" library="supply1" deviceset="GND" device=""/>
@@
 <part name="J7" library="con-amp" deviceset="MTA04-100" device=""/>
 <part name="GND10" library="supply1" deviceset="GND" device=""/>
-<part name="R7" library="resistor" deviceset="R-EU_" device="0207/7"/>
-<part name="R8" library="resistor" deviceset="R-EU_" device="0207/7"/>
+<part name="R7" library="resistor" deviceset="R-EU_" device="0207/7" value="4K7"/>
+<part name="R8" library="resistor" deviceset="R-EU_" device="0207/7" value="4K7"/>
 <part name="PAD9" library="wirepad" deviceset="WIREPAD" device="1,6/0,9" value="WIREPAD1,6/0,9"/>
 <part name="PAD10" library="wirepad" deviceset="WIREPAD" device="1,6/0,9" value="WIREPAD1,6/0,9"/>
@@
 <attribute name="VALUE" x="58.928" y="112.522" size="1.778" layer="96" rot="R180"/>
 </instance>
-<instance part="R1" gate="G$1" x="182.245" y="55.88"/>
-<instance part="R2" gate="G$1" x="182.245" y="50.8"/>
-<instance part="R3" gate="G$1" x="182.88" y="44.45"/>
-<instance part="R4" gate="G$1" x="182.88" y="40.005"/>
-<instance part="R5" gate="G$1" x="182.88" y="34.925"/>
-<instance part="R6" gate="G$1" x="182.88" y="30.48"/>
+<instance part="R1" gate="G$1" x="182.245" y="55.88" smashed="yes">
+<attribute name="NAME" x="178.435" y="57.3786" size="1.778" layer="95"/>
+<attribute name="VALUE" x="180.34" y="55.118" size="1.778" layer="96"/>
+</instance>
+<instance part="R2" gate="G$1" x="182.245" y="50.8" smashed="yes">
+<attribute name="NAME" x="178.435" y="52.2986" size="1.778" layer="95"/>
+<attribute name="VALUE" x="180.34" y="50.038" size="1.778" layer="96"/>
+</instance>
+<instance part="R3" gate="G$1" x="182.88" y="44.45" smashed="yes">
+<attribute name="NAME" x="179.07" y="45.9486" size="1.778" layer="95"/>
+<attribute name="VALUE" x="180.975" y="43.688" size="1.778" layer="96"/>
+</instance>
+<instance part="R4" gate="G$1" x="182.88" y="40.005" smashed="yes">
+<attribute name="NAME" x="179.07" y="41.5036" size="1.778" layer="95"/>
+<attribute name="VALUE" x="180.975" y="39.243" size="1.778" layer="96"/>
+</instance>
+<instance part="R5" gate="G$1" x="182.88" y="34.925" smashed="yes">
+<attribute name="NAME" x="178.435" y="36.4236" size="1.778" layer="95"/>
+<attribute name="VALUE" x="180.975" y="34.163" size="1.778" layer="96"/>
+</instance>
+<instance part="R6" gate="G$1" x="182.88" y="30.48" smashed="yes">
+<attribute name="NAME" x="179.07" y="31.9786" size="1.778" layer="95"/>
+<attribute name="VALUE" x="180.975" y="29.718" size="1.778" layer="96"/>
+</instance>
 <instance part="GND7" gate="1" x="175.26" y="30.48" rot="R270"/>
 <instance part="GND8" gate="1" x="174.625" y="50.8" rot="R270"/>
@@
 </instance>
 <instance part="GND10" gate="1" x="90.17" y="84.455" rot="R90"/>
-<instance part="R7" gate="G$1" x="80.645" y="92.075" rot="R90"/>
-<instance part="R8" gate="G$1" x="84.455" y="94.615" rot="R90"/>
+<instance part="R7" gate="G$1" x="80.645" y="92.075" smashed="yes" rot="R90">
+<attribute name="NAME" x="79.375" y="96.2914" size="1.778" layer="95" rot="R180"/>
+<attribute name="VALUE" x="81.407" y="89.535" size="1.778" layer="96" rot="R90"/>
+</instance>
+<instance part="R8" gate="G$1" x="84.455" y="94.615" smashed="yes" rot="R90">
+<attribute name="NAME" x="89.535" y="96.2914" size="1.778" layer="95" rot="R180"/>
+<attribute name="VALUE" x="83.693" y="97.155" size="1.778" layer="96" rot="R270"/>
+</instance>
 <instance part="PAD9" gate="G$1" x="20.32" y="126.365" smashed="yes">
 <attribute name="NAME" x="12.192" y="125.6792" size="1.778" layer="95"/>
@@
 <net name="ENAM1" class="0">
 <segment>
-<pinref part="J4" gate="G$1" pin="4"/>
-<wire x1="77.47" y1="41.91" x2="79.375" y2="41.91" width="0.1524" layer="91"/>
-<label x="79.375" y="41.91" size="1.778" layer="95" xref="yes"/>
-</segment>
-<segment>
 <pinref part="IC1" gate="G$1" pin="1-2EN"/>
 <wire x1="142.875" y1="23.495" x2="144.145" y2="23.495" width="0.1524" layer="91"/>
@@
 <wire x1="25.4" y1="109.22" x2="24.13" y2="109.22" width="0.1524" layer="91"/>
 <label x="24.13" y="109.22" size="1.778" layer="95" rot="R180" xref="yes"/>
+</segment>
+<segment>
+<pinref part="J4" gate="G$1" pin="2"/>
+<wire x1="77.47" y1="36.83" x2="79.375" y2="36.83" width="0.1524" layer="91"/>
+<label x="79.375" y="36.83" size="1.778" layer="95" xref="yes"/>
 </segment>
 </net>
@@
 </segment>
 </net>
-<net name="AUX2" class="0">
+<net name="AUX3" class="0">
 <segment>
 <pinref part="J1" gate="G$2" pin="9"/>
@@
 </segment>
 </net>
+<net name="AUX1/TX2" class="0">
+<segment>
+<pinref part="J4" gate="G$1" pin="4"/>
+<wire x1="77.47" y1="41.91" x2="78.105" y2="41.91" width="0.1524" layer="91"/>
+<label x="78.74" y="41.91" size="1.778" layer="95" xref="yes"/>
+</segment>
+<segment>
+<pinref part="X4" gate="-1" pin="KL"/>
+<wire x1="191.135" y1="116.84" x2="192.405" y2="116.84" width="0.1524" layer="91"/>
+<label x="192.405" y="116.84" size="1.778" layer="95" xref="yes"/>
+</segment>
+</net>
+<net name="AUX2/RX2" class="0">
+<segment>
+<pinref part="J4" gate="G$1" pin="3"/>
+<wire x1="77.47" y1="39.37" x2="78.105" y2="39.37" width="0.1524" layer="91"/>
+<label x="78.105" y="39.37" size="1.778" layer="95" xref="yes"/>
+</segment>
+<segment>
+<pinref part="X4" gate="-2" pin="KL"/>
+<wire x1="191.135" y1="111.76" x2="192.405" y2="111.76" width="0.1524" layer="91"/>
+<label x="193.04" y="111.76" size="1.778" layer="95" xref="yes"/>
+</segment>
+</net>
