File: Robotec/MUBI-BOT/mubi-bot-3.sch (EAGLE design)
At the start: 8 parts, among them IC1 L293E

Commit message: update MUBI-BOT
Parts:
- added PAD1, PAD2: WIREPAD1,6/0,9, wirepad:WIREPAD1,6/0,9
Connections:
- net +5V: now also IC1.VCC1, PAD1.P, PAD2.P
- net VBAT: no longer IC1.VCC1
Other:
- note added: "PLACA ROBOT ARDUINO NANO"
- moved on the sheet: C1, C2
Changed lines of the file:
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@@
 <setting verticaltext="up"/>
 </settings>
-<grid distance="25" unitdist="mil" unit="mil" style="lines" multiple="1" display="yes" altdistance="0.01" altunitdist="inch" altunit="inch"/>
+<grid distance="0.1" unitdist="inch" unit="inch" style="lines" multiple="1" display="no" altdistance="0.01" altunitdist="inch" altunit="inch"/>
 <layers>
 <layer number="1" name="Top" color="4" fill="1" visible="no" active="no"/>
@@
 <part name="SUPPLY3" library="supply2" deviceset="+5V" device=""/>
 <part name="GND8" library="supply1" deviceset="GND" device=""/>
+<part name="PAD1" library="wirepad" deviceset="WIREPAD" device="1,6/0,9"/>
+<part name="PAD2" library="wirepad" deviceset="WIREPAD" device="1,6/0,9"/>
+<part name="SUPPLY4" library="supply2" deviceset="+5V" device=""/>
 </parts>
 <sheets>
 <sheet>
 <plain>
+<text x="66.04" y="106.68" size="2.54" layer="91">PLACA ROBOT ARDUINO NANO</text>
 </plain>
 <instances>
@@
 <instance part="GND4" gate="1" x="31.75" y="51.435" rot="R270"/>
 <instance part="GND1" gate="1" x="79.375" y="56.515" rot="R90"/>
-<instance part="SUPPLY1" gate="+5V" x="88.9" y="53.975"/>
+<instance part="SUPPLY1" gate="+5V" x="85.725" y="53.975"/>
 <instance part="X1" gate="-1" x="26.67" y="96.52"/>
 <instance part="X1" gate="-2" x="26.67" y="91.44"/>
@@
 <instance part="SUPPLY2" gate="+5V" x="147.32" y="65.405" rot="R270"/>
 <instance part="GND5" gate="1" x="155.575" y="67.945" rot="R90"/>
-<instance part="C1" gate="G$1" x="88.9" y="48.895"/>
-<instance part="C2" gate="G$1" x="95.25" y="56.515"/>
-<instance part="GND6" gate="1" x="88.9" y="41.275"/>
-<instance part="GND7" gate="1" x="95.25" y="48.895"/>
+<instance part="C1" gate="G$1" x="165.735" y="46.99" smashed="yes">
+<attribute name="NAME" x="167.259" y="42.926" size="1.778" layer="95"/>
+<attribute name="VALUE" x="167.259" y="42.291" size="1.778" layer="96"/>
+</instance>
+<instance part="C2" gate="G$1" x="92.075" y="56.515"/>
+<instance part="GND6" gate="1" x="165.735" y="39.37"/>
+<instance part="GND7" gate="1" x="92.075" y="48.26"/>
 <instance part="S1" gate="1" x="15.24" y="31.115" smashed="yes" rot="R90">
 <attribute name="NAME" x="5.715" y="34.29" size="1.778" layer="95" rot="R180"/>
@@
 <instance part="SUPPLY3" gate="+5V" x="10.16" y="37.465"/>
 <instance part="GND8" gate="1" x="10.16" y="22.225"/>
+<instance part="PAD1" gate="G$1" x="106.045" y="8.89" smashed="yes">
+<attribute name="NAME" x="97.917" y="8.2042" size="1.778" layer="95"/>
+<attribute name="VALUE" x="104.902" y="5.588" size="1.778" layer="96"/>
+</instance>
+<instance part="PAD2" gate="G$1" x="171.45" y="50.165" smashed="yes" rot="R180">
+<attribute name="NAME" x="179.578" y="50.8508" size="1.778" layer="95" rot="R180"/>
+<attribute name="VALUE" x="186.563" y="54.102" size="1.778" layer="96" rot="R180"/>
+</instance>
+<instance part="SUPPLY4" gate="+5V" x="165.735" y="55.88"/>
 </instances>
 <busses>
@@
 <pinref part="C2" gate="G$1" pin="-"/>
 <pinref part="GND7" gate="1" pin="GND"/>
+<wire x1="92.075" y1="51.435" x2="92.075" y2="50.8" width="0.1524" layer="91"/>
 </segment>
 <segment>
@@
 <segment>
 <pinref part="ARDUINO_NANO1" gate="G$1" pin="VIN"/>
-<wire x1="75.565" y1="59.055" x2="95.25" y2="59.055" width="0.1524" layer="91"/>
+<wire x1="75.565" y1="59.055" x2="92.075" y2="59.055" width="0.1524" layer="91"/>
 <label x="97.79" y="59.055" size="1.778" layer="95" xref="yes"/>
 <pinref part="C2" gate="G$1" pin="+"/>
-<wire x1="95.25" y1="59.055" x2="97.79" y2="59.055" width="0.1524" layer="91"/>
-<junction x="95.25" y="59.055"/>
+<wire x1="92.075" y1="59.055" x2="97.79" y2="59.055" width="0.1524" layer="91"/>
+<junction x="92.075" y="59.055"/>
 </segment>
 <segment>
@@
 </segment>
 <segment>
-<pinref part="IC1" gate="G$1" pin="VCC1"/>
-<wire x1="111.125" y1="13.335" x2="110.49" y2="13.335" width="0.1524" layer="91"/>
-<label x="110.49" y="13.335" size="1.778" layer="95" rot="R180" xref="yes"/>
-</segment>
-<segment>
 <pinref part="IC1" gate="G$1" pin="VCC2"/>
 <wire x1="141.605" y1="48.895" x2="142.24" y2="48.895" width="0.1524" layer="91"/>
@@
 <net name="+5V" class="0">
 <segment>
-<pinref part="ARDUINO_NANO1" gate="G$1" pin="5V"/>
-<wire x1="75.565" y1="51.435" x2="88.9" y2="51.435" width="0.1524" layer="91"/>
-<pinref part="SUPPLY1" gate="+5V" pin="+5V"/>
-<pinref part="C1" gate="G$1" pin="1"/>
-<junction x="88.9" y="51.435"/>
-</segment>
-<segment>
 <pinref part="X2" gate="-3" pin="KL"/>
 <wire x1="92.71" y1="86.36" x2="93.98" y2="86.36" width="0.1524" layer="91"/>
@@
 <wire x1="10.16" y1="34.925" x2="10.16" y2="33.655" width="0.1524" layer="91"/>
 </segment>
-</net>
+<segment>
+<pinref part="ARDUINO_NANO1" gate="G$1" pin="5V"/>
+<pinref part="SUPPLY1" gate="+5V" pin="+5V"/>
+<wire x1="75.565" y1="51.435" x2="85.725" y2="51.435" width="0.1524" layer="91"/>
+</segment>
+<segment>
+<pinref part="SUPPLY4" gate="+5V" pin="+5V"/>
+<pinref part="C1" gate="G$1" pin="1"/>
+<wire x1="165.735" y1="49.53" x2="165.735" y2="50.165" width="0.1524" layer="91"/>
+<pinref part="PAD2" gate="G$1" pin="P"/>
+<wire x1="165.735" y1="50.165" x2="165.735" y2="53.34" width="0.1524" layer="91"/>
+<wire x1="168.91" y1="50.165" x2="165.735" y2="50.165" width="0.1524" layer="91"/>
+</segment>
+<segment>
+<pinref part="IC1" gate="G$1" pin="VCC1"/>
+<wire x1="111.125" y1="13.335" x2="106.045" y2="13.335" width="0.1524" layer="91"/>
+<wire x1="111.125" y1="13.335" x2="111.125" y2="8.89" width="0.1524" layer="91"/>
+<wire x1="111.125" y1="8.89" x2="108.585" y2="8.89" width="0.1524" layer="91"/>
+<pinref part="PAD1" gate="G$1" pin="P"/>
+<label x="105.41" y="13.335" size="1.778" layer="95" rot="R180" xref="yes"/>
+</segment>
+</net>

Commit message: update MUBI-BOT
Other:
- note removed: "PLACA ROBOT ARDUINO NANO"
Changed lines of the file:
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@@
 <sheet>
 <plain>
-<text x="66.04" y="106.68" size="2.54" layer="91">PLACA ROBOT ARDUINO NANO</text>
 </plain>
 <instances>

Commit message: update sch & brd
Parts:
- added D1: 1N4004, diode:1N4004
- added H1, H2: MOUNT-HOLE2.8, holes:MOUNT-HOLE2.8
- added PAD3, PAD4, PAD5, PAD6, PAD7, PAD8: WIREPAD1,6/0,9, wirepad:WIREPAD1,6/0,9
Connections:
- removed net VBAT: ARDUINO_NANO1.VIN, C2.+, IC1.VCC2, X2-1.KL
- new net +VBAT: D1.A, X2-1.KL
- new net +VCC: ARDUINO_NANO1.VIN, C2.+, D1.C, IC1.VCC2, PAD3.P, PAD4.P
- net GND: now also PAD5.P, PAD6.P, PAD7.P, PAD8.P
Other:
- note added: "PLACA ROBOT ARDUINO NANO"
- moved on the sheet: SV1, X1-1, X1-2, X1-3, X1-4, X1-5, X2-10, X2-6, X2-7, X2-8, X2-9

Commit message: update mubi-bot
Parts:
- removed D1: 1N4004, diode:1N4004
- removed H1, H2: MOUNT-HOLE2.8, holes:MOUNT-HOLE2.8
- removed PAD3, PAD4, PAD5, PAD6, PAD7, PAD8: WIREPAD1,6/0,9, wirepad:WIREPAD1,6/0,9
Connections:
- removed net +VCC: ARDUINO_NANO1.VIN, C2.+, D1.C, IC1.VCC2, PAD3.P, PAD4.P
- net +VBAT: now also ARDUINO_NANO1.VIN, C2.+, IC1.VCC2; no longer D1.A
- net GND: no longer PAD5.P, PAD6.P, PAD7.P, PAD8.P
