File: Robotec/MUBI-BOT/mubi-bot-3/mubi-bot-3.kicad_sch (KiCad schematic)
At the start: 10 parts, among them IC1 L293E, X1 AK500/10-H, X2 AK500/10-H

Commit message: update sch pcb kicad v9
Parts:
- IC1: value L293E -> L293D
- renumbered ARDUINO_NANO1 to ARDUINO_NANO
Connections:
- no-connect marks 0 -> 9
Other:
- note removed: "PLACA ROBOT ARDUINO NANO"
- company: (none) -> E.E.S.T. N.°5 "AMANCIO WILLIAMS"
- title: (none) -> MUBI-BOT NANO v4
- moved on the sheet: ARDUINO_NANO, C1, C2, IC1, PAD1, PAD2, S1, SV1, X1A, X1B, X1C, X1D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

Commit message: update sch & pcb
Parts:
- removed S1: 9450-1, mubi-bot-3:9450-1, symbol mubi-bot-3-eagle-import:9450-1
- added J1: SEL, Connector_PinHeader_2.54mm:PinHeader_1x03_P2.54mm_Vertical, symbol Connector:Conn_01x03_Pin
Connections:
- net +5V: now also J1.1 (Pin_1)
- net GND: now also J1.3 (Pin_3)
- net at ARDUINO_NANO.27 (D9/OC1A): now also J1.2 (Pin_2)
Other:
- title: MUBI-BOT NANO v4 -> MUBI-BOT NANO
Changed lines of the file:
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@@
 	(paper "A4")
 	(title_block
-		(title "MUBI-BOT NANO v4")
+		(title "MUBI-BOT NANO")
 		(date "2025-07-16")
-		(rev "1.0")
+		(rev "4.0")
 		(company "E.E.S.T. N.°5 \"AMANCIO WILLIAMS\"")
 		(comment 1 "Diseño Original: Prof. Ing. Fermín Oyarburo")
@@
 	(wire
 		(pts
-			(xy 72.39 106.68) (xy 77.47 106.68)
-		)
-		(stroke
-			(width 0.1524)
-			(type solid)
-		)
-	)
-	(wire
-		(pts
 			(xy 99.06 60.96) (xy 106.68 60.96)
 		)
@@
 	(wire
 		(pts
-			(xy 180.34 129.54) (xy 173.99 129.54)
+			(xy 57.15 129.54) (xy 58.42 129.54)
 		)
 		(stroke
-			(width 0.1524)
-			(type solid)
+			(width 0)
+			(type default)
 		)
 	)
 	(wire
 		(pts
-			(xy 77.47 111.76) (xy 69.85 111.76)
+			(xy 180.34 129.54) (xy 173.99 129.54)
 		)
 		(stroke
@@
 	(wire
 		(pts
-			(xy 118.11 114.3) (xy 125.73 114.3)
+			(xy 77.47 111.76) (xy 69.85 111.76)
 		)
 		(stroke
@@
 	(wire
 		(pts
-			(xy 52.705 123.19) (xy 52.705 124.46)
+			(xy 118.11 114.3) (xy 125.73 114.3)
 		)
 		(stroke
@@
 	(wire
 		(pts
+			(xy 58.42 124.46) (xy 57.15 124.46)
+		)
+		(stroke
+			(width 0)
+			(type default)
+		)
+	)
+	(wire
+		(pts
 			(xy 77.47 119.38) (xy 69.85 119.38)
 		)
@@
 	(wire
 		(pts
+			(xy 58.42 121.92) (xy 58.42 124.46)
+		)
+		(stroke
+			(width 0)
+			(type default)
+		)
+	)
+	(wire
+		(pts
+			(xy 57.15 127) (xy 77.47 127)
+		)
+		(stroke
+			(width 0)
+			(type default)
+		)
+	)
+	(wire
+		(pts
 			(xy 180.34 124.46) (xy 173.99 124.46)
 		)
@@
 	(wire
 		(pts
-			(xy 60.96 104.14) (xy 72.39 104.14)
+			(xy 69.85 106.68) (xy 77.47 106.68)
 		)
 		(stroke
@@
 	(wire
 		(pts
-			(xy 52.705 133.35) (xy 52.705 129.54)
+			(xy 200.66 49.53) (xy 200.66 60.96)
 		)
 		(stroke
@@
 	(wire
 		(pts
-			(xy 200.66 49.53) (xy 200.66 60.96)
+			(xy 58.42 129.54) (xy 58.42 132.08)
 		)
 		(stroke
-			(width 0.1524)
-			(type solid)
+			(width 0)
+			(type default)
 		)
 	)
@@
 	(wire
 		(pts
-			(xy 72.39 104.14) (xy 72.39 106.68)
-		)
-		(stroke
-			(width 0.1524)
-			(type solid)
-		)
-	)
-	(wire
-		(pts
 			(xy 210.82 124.46) (xy 217.17 124.46)
 		)
@@
 	(wire
 		(pts
-			(xy 77.47 127) (xy 62.865 127)
-		)
-		(stroke
-			(width 0.1524)
-			(type solid)
-		)
-	)
-	(wire
-		(pts
 			(xy 213.36 116.84) (xy 214.63 116.84)
 		)
@@
 		)
 	)
+	(label "GND"
+		(at 69.85 106.68 0)
+		(effects
+			(font
+				(size 1.2446 1.2446)
+			)
+			(justify left bottom)
+		)
+	)
 	(label "INFRA1"
 		(at 69.85 111.76 0)
@@
 	)
 	(symbol
+		(lib_id "Connector:Conn_01x03_Pin")
+		(at 52.07 127 0)
+		(unit 1)
+		(exclude_from_sim no)
+		(in_bom yes)
+		(on_board yes)
+		(dnp no)
+		(property "Reference" "J1"
+			(at 50.292 120.396 0)
+			(effects
+				(font
+					(size 1.27 1.27)
+				)
+			)
+		)
+		(property "Value" "SEL"
+			(at 50.8 122.174 0)
+			(effects
+				(font
+					(size 1.27 1.27)
+				)
+			)
+		)
+		(property "Footprint" "Connector_PinHeader_2.54mm:PinHeader_1x03_P2.54mm_Vertical"
+			(at 52.07 127 0)
+			(effects
+				(font
+					(size 1.27 1.27)
+				)
+				(hide yes)
+			)
+		)
+		(property "Datasheet" "~"
+			(at 52.07 127 0)
+			(effects
+				(font
+					(size 1.27 1.27)
+				)
+				(hide yes)
+			)
+		)
+		(property "Description" "Generic connector, single row, 01x03, script generated"
+			(at 52.07 127 0)
+			(effects
+				(font
+					(size 1.27 1.27)
+				)
+				(hide yes)
+			)
+		)
+		(pin "2"
+		)
+		(pin "1"
+		)
+		(pin "3"
+		)
+		(instances
+			(project ""
+				(path "/a0797d60-6025-4c6e-a7a0-fe437631a5ca"
+					(reference "J1")
+					(unit 1)
+				)
+			)
+		)
+	)
+	(symbol
 		(lib_id "mubi-bot-3-eagle-import:GND")
 		(at 173.99 116.84 270)
@@
 	(symbol
 		(lib_id "mubi-bot-3-eagle-import:GND")
-		(at 52.705 135.89 0)
+		(at 58.42 134.62 0)
 		(unit 1)
 		(exclude_from_sim no)
@@
 		(dnp no)
 		(property "Reference" "#GND8"
-			(at 52.705 135.89 0)
+			(at 58.42 134.62 0)
 			(effects
 				(font
@@
 		)
 		(property "Value" "GND"
-			(at 50.165 138.43 0)
+			(at 55.88 137.16 0)
 			(effects
 				(font
@@
 		)
 		(property "Footprint" ""
-			(at 52.705 135.89 0)
+			(at 58.42 134.62 0)
 			(effects
 				(font
@@
 		)
 		(property "Datasheet" ""
-			(at 52.705 135.89 0)
+			(at 58.42 134.62 0)
 			(effects
 				(font
@@
 		)
 		(property "Description" ""
-			(at 52.705 135.89 0)
+			(at 58.42 134.62 0)
 			(effects
 				(font
@@
 	(symbol
 		(lib_id "mubi-bot-3-eagle-import:+5V")
-		(at 52.705 120.65 0)
+		(at 58.42 119.38 0)
 		(unit 1)
 		(exclude_from_sim no)
@@
 		(dnp no)
 		(property "Reference" "#SUPPLY3"
-			(at 52.705 120.65 0)
+			(at 58.42 119.38 0)
 			(effects
 				(font
@@
 		)
 		(property "Value" "+5V"
-			(at 50.8 117.475 0)
+			(at 56.515 116.205 0)
 			(effects
 				(font
@@
 		)
 		(property "Footprint" ""
-			(at 52.705 120.65 0)
+			(at 58.42 119.38 0)
 			(effects
 				(font
@@
 		)
 		(property "Datasheet" ""
-			(at 52.705 120.65 0)
+			(at 58.42 119.38 0)
 			(effects
 				(font
@@
 		)
 		(property "Description" ""
-			(at 52.705 120.65 0)
+			(at 58.42 119.38 0)
 			(effects
 				(font
@@
 	)
 	(symbol
-		(lib_id "mubi-bot-3-eagle-import:GND")
-		(at 58.42 104.14 270)
-		(unit 1)
-		(exclude_from_sim no)
-		(in_bom yes)
-		(on_board yes)
-		(dnp no)
-		(property "Reference" "#GND4"
-			(at 58.42 104.14 0)
-			(effects
-				(font
-					(size 1.27 1.27)
-				)
-				(hide yes)
-			)
-		)
-		(property "Value" "GND"
-			(at 55.88 101.6 0)
-			(effects
-				(font
-					(size 1.778 1.5113)
-				)
-				(justify left bottom)
-			)
-		)
-		(property "Footprint" ""
-			(at 58.42 104.14 0)
-			(effects
-				(font
-					(size 1.27 1.27)
-				)
-				(hide yes)
-			)
-		)
-		(property "Datasheet" ""
-			(at 58.42 104.14 0)
-			(effects
-				(font
-					(size 1.27 1.27)
-				)
-				(hide yes)
-			)
-		)
-		(property "Description" ""
-			(at 58.42 104.14 0)
-			(effects
-				(font
-					(size 1.27 1.27)
-				)
-				(hide yes)
-			)
-		)
-		(pin "1"
-		)
-		(instances
-			(project ""
-				(path "/a0797d60-6025-4c6e-a7a0-fe437631a5ca"
-					(reference "#GND4")
-					(unit 1)
-				)
-			)
-		)
-	)
-	(symbol
 		(lib_id "mubi-bot-3-eagle-import:AK500/10-H")
 		(at 69.85 45.72 0)
@@
 					(unit 1)
 				)
-			)
-		)
-	)
-	(symbol
-		(lib_id "mubi-bot-3-eagle-import:9450-1")
-		(at 57.785 127 90)
-		(unit 1)
-		(exclude_from_sim no)
-		(in_bom yes)
-		(on_board yes)
-		(dnp no)
-		(property "Reference" "S1"
-			(at 48.26 123.825 90)
-			(effects
-				(font
-					(size 1.778 1.5113)
-				)
-				(justify left bottom)
-			)
-		)
-		(property "Value" "9450-1"
-			(at 52.07 126.365 90)
-			(effects
-				(font
-					(size 1.778 1.5113)
-				)
-				(justify left bottom)
-			)
-		)
-		(property "Footprint" "mubi-bot-3:9450-1"
-			(at 57.785 127 0)
-			(effects
-				(font
-					(size 1.27 1.27)
-				)
-				(hide yes)
-			)
-		)
-		(property "Datasheet" ""
-			(at 57.785 127 0)
-			(effects
-				(font
-					(size 1.27 1.27)
-				)
-				(hide yes)
-			)
-		)
-		(property "Description" ""
-			(at 57.785 127 0)
-			(effects
-				(font
-					(size 1.27 1.27)
-				)
-				(hide yes)
-			)
-		)
-		(pin "1"
-		)
-		(pin "2"
-		)
-		(pin "3"
-		)
-		(instances
-			(project ""
-				(path "/a0797d60-6025-4c6e-a7a0-fe437631a5ca"
-					(reference "S1")
-					(unit 1)
-				)

Commit message: update sch&pcb&step
Parts:
- added H1, H2: MountingHole, MountingHole:MountingHole_2.2mm_M2, symbol Mechanical:MountingHole
- renumbered ARDUINO_NANO to ARDUINO_NANO1
Changed lines of the file:
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@@
 		(on_board yes)
 		(dnp no)
-		(property "Reference" "ARDUINO_NANO"
+		(property "Reference" "ARDUINO_NANO1"
 			(at 82.55 94.742 0)
 			(effects
@@
 			(project ""
 				(path "/a0797d60-6025-4c6e-a7a0-fe437631a5ca"
-					(reference "ARDUINO_NANO")
+					(reference "ARDUINO_NANO1")
 					(unit 1)
 				)
@@
 	)
 	(symbol
+		(lib_id "Mechanical:MountingHole")
+		(at 241.3 104.14 0)
+		(unit 1)
+		(exclude_from_sim no)
+		(in_bom no)
+		(on_board yes)
+		(dnp no)
+		(fields_autoplaced yes)
+		(property "Reference" "H2"
+			(at 243.84 102.8699 0)
+			(effects
+				(font
+					(size 1.27 1.27)
+				)
+				(justify left)
+			)
+		)
+		(property "Value" "MountingHole"
+			(at 243.84 105.4099 0)
+			(effects
+				(font
+					(size 1.27 1.27)
+				)
+				(justify left)
+				(hide yes)
+			)
+		)
+		(property "Footprint" "MountingHole:MountingHole_2.2mm_M2"
+			(at 241.3 104.14 0)
+			(effects
+				(font
+					(size 1.27 1.27)
+				)
+				(hide yes)
+			)
+		)
+		(property "Datasheet" "~"
+			(at 241.3 104.14 0)
+			(effects
+				(font
+					(size 1.27 1.27)
+				)
+				(hide yes)
+			)
+		)
+		(property "Description" "Mounting Hole without connection"
+			(at 241.3 104.14 0)
+			(effects
+				(font
+					(size 1.27 1.27)
+				)
+				(hide yes)
+			)
+		)
+		(instances
+			(project "mubi-bot-3"
+				(path "/a0797d60-6025-4c6e-a7a0-fe437631a5ca"
+					(reference "H2")
+					(unit 1)
+				)
+			)
+		)
+	)
+	(symbol
 		(lib_id "mubi-bot-3-eagle-import:MA05-1")
 		(at 190.5 55.88 0)
@@
 					(unit 1)
 				)
+			)
+		)
+	)
+	(symbol
+		(lib_id "Mechanical:MountingHole")
+		(at 241.3 99.06 0)
+		(unit 1)
+		(exclude_from_sim no)
+		(in_bom no)
+		(on_board yes)
+		(dnp no)
+		(fields_autoplaced yes)
+		(property "Reference" "H1"
+			(at 243.84 97.7899 0)
+			(effects
+				(font
+					(size 1.27 1.27)
+				)
+				(justify left)
+			)
+		)
+		(property "Value" "MountingHole"
+			(at 243.84 100.3299 0)
+			(effects
+				(font
+					(size 1.27 1.27)
+				)
+				(justify left)
+				(hide yes)
+			)
+		)
+		(property "Footprint" "MountingHole:MountingHole_2.2mm_M2"
+			(at 241.3 99.06 0)
+			(effects
+				(font
+					(size 1.27 1.27)
+				)
+				(hide yes)
+			)
+		)
+		(property "Datasheet" "~"
+			(at 241.3 99.06 0)
+			(effects
+				(font
+					(size 1.27 1.27)
+				)
+				(hide yes)
+			)
+		)
+		(property "Description" "Mounting Hole without connection"
+			(at 241.3 99.06 0)
+			(effects
+				(font
+					(size 1.27 1.27)
+				)
+				(hide yes)
+			)
+		)
+		(instances
+			(project ""
+				(path "/a0797d60-6025-4c6e-a7a0-fe437631a5ca"
+					(reference "H1")
+					(unit 1)
+				)
