File: Robotec/MUBI-BOT/mubi-bot-3/mubi-bot-3.kicad_pcb (KiCad board)
At the start: 2 copper layers, 49.8 x 50.8 mm, 10 parts, among them IC1 L293E

Commit message: update sch pcb kicad v9
Other:
- board text removed: "mascara de agujeros"

Commit message: update sch & pcb
Parts:
- removed S1: 9450-1, mubi-bot-3:9450-1
- added J1: SEL, Connector_PinHeader_2.54mm:PinHeader_1x03_P2.54mm_Vertical, F.Cu at (141.0, 82.5)
- ARDUINO_NANO1: value (none) -> ARDUINO_NANO
- C1: value (none) -> C-EU050-025X075
- C2: value (none) -> CPOL-EUE2.5-5
- IC1: value L293E -> L293D
- SV1: value (none) -> MA05-1
- X1, X2: value (none) -> AK500/10-H
Connections:
- net +VBAT renamed /+VBAT
- net AUX1 renamed /AUX1
- net AUX2 renamed /AUX2
- net CM11 renamed /CM11
- net CM12 renamed /CM12
- net CM21 renamed /CM21
- net CM22 renamed /CM22
- net ECHO1 renamed /ECHO1
- net ECHO2 renamed /ECHO2
- net ECHO3 renamed /ECHO3
- net ENA1 renamed /ENA1
- net ENA2 renamed /ENA2
- net INFRA1 renamed /INFRA1
- net INFRA2 renamed /INFRA2
- net INFRA3 renamed /INFRA3
- net M1A renamed /M1A
- net M1B renamed /M1B
- net M2A renamed /M2A
- net M2B renamed /M2B
- net SCL renamed /SCL
- net SDA renamed /SDA
- net TRIG renamed /TRIG
- ARDUINO_NANO1 pad 10: (no net) -> unconnected-(ARDUINO_NANO1-ADC6/A6-Pad10)
- ARDUINO_NANO1 pad 11: (no net) -> unconnected-(ARDUINO_NANO1-ADC7/A7-Pad11)
- ARDUINO_NANO1 pad 13: (no net) -> unconnected-(ARDUINO_NANO1-~{RESET@2}-Pad13)
- ARDUINO_NANO1 pad 16: (no net) -> unconnected-(ARDUINO_NANO1-D1/TX-Pad16)
- ARDUINO_NANO1 pad 17: (no net) -> unconnected-(ARDUINO_NANO1-D0/RX-Pad17)
- ARDUINO_NANO1 pad 18: (no net) -> unconnected-(ARDUINO_NANO1-~{RESET@1}-Pad18)
- ARDUINO_NANO1 pad 2: (no net) -> unconnected-(ARDUINO_NANO1-3V3-Pad2)
- ARDUINO_NANO1 pad 3: (no net) -> unconnected-(ARDUINO_NANO1-AREF-Pad3)
- IC1 pad 4: N$1 -> GND
- IC1 pad 5: N$1 -> GND
- SV1 pad 5: (no net) -> unconnected-(SV1-Pad5)
Routing:
- net N$1: track 5.61 -> 0.00 mm, vias 1 -> 0
- net GND: track 187.0 -> 191.1 mm, vias 3 -> 4
- net Net-(ARDUINO_NANO1-D9/OC1A): track 48.8 -> 47.3 mm
- net +5V: track 110.0 -> 109.3 mm
Other:
- board text added: "+VBAT"
- board text removed: "+ VBAT"

Commit message: update sch&pcb&step
Parts:
- added H1: MountingHole, MountingHole:MountingHole_2.2mm_M2, F.Cu at (134.6, 86.4)
- added H2: MountingHole, MountingHole:MountingHole_2.2mm_M2, F.Cu at (161.3, 123.2)
Routing:
- net Net-(ARDUINO_NANO1-D9/OC1A): track 47.3 -> 44.7 mm
Changed lines of the file:
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@@
+		(embedded_fonts no)
+	)
+	(footprint "MountingHole:MountingHole_2.2mm_M2"
+		(layer "F.Cu")
+		(at 134.62 86.36)
+		(descr "Mounting Hole 2.2mm, M2, no annular, generated by kicad-footprint-generator mountinghole.py")
+		(tags "mountinghole M2")
+		(property "Reference" "H1"
+			(at 0 -3.15 0)
+			(layer "F.SilkS")
+			(hide yes)
+			(effects
+				(font
+					(size 1 1)
+					(thickness 0.15)
+				)
+			)
+		)
+		(property "Value" "MountingHole"
+			(at 0 3.15 0)
+			(layer "F.Fab")
+			(hide yes)
+			(effects
+				(font
+					(size 1 1)
+					(thickness 0.15)
+				)
+			)
+		)
+		(property "Datasheet" "~"
+			(at 0 0 0)
+			(layer "F.Fab")
+			(hide yes)
+			(effects
+				(font
+					(size 1.27 1.27)
+					(thickness 0.15)
+				)
+			)
+		)
+		(property "Description" "Mounting Hole without connection"
+			(at 0 0 0)
+			(layer "F.Fab")
+			(hide yes)
+			(effects
+				(font
+					(size 1.27 1.27)
+					(thickness 0.15)
+				)
+			)
+		)
+		(property ki_fp_filters "MountingHole*")
+		(sheetname "/")
+		(sheetfile "mubi-bot-3.kicad_sch")
+		(attr exclude_from_pos_files exclude_from_bom)
+		(fp_circle
+			(center 0 0)
+			(end 2.2 0)
+			(stroke
+				(width 0.15)
+				(type solid)
+			)
+			(fill no)
+			(layer "Cmts.User")
+		)
+		(fp_circle
+			(center 0 0)
+			(end 2.45 0)
+			(stroke
+				(width 0.05)
+				(type solid)
+			)
+			(fill no)
+			(layer "F.CrtYd")
+		)
+		(fp_text user "${REFERENCE}"
+			(at 0 0 0)
+			(layer "F.Fab")
+			(effects
+				(font
+					(size 1 1)
+					(thickness 0.15)
+				)
+			)
+		)
+		(pad "" np_thru_hole circle
+			(at 0 0)
+			(size 2.2 2.2)
+			(drill 2.2)
+			(layers "*.Cu" "*.Mask")
+		)
+		(embedded_fonts no)
+	)
+	(footprint "MountingHole:MountingHole_2.2mm_M2"
+		(layer "F.Cu")
+		(at 161.29 123.19)
+		(descr "Mounting Hole 2.2mm, M2, no annular, generated by kicad-footprint-generator mountinghole.py")
+		(tags "mountinghole M2")
+		(property "Reference" "H2"
+			(at 0 -3.15 0)
+			(layer "F.SilkS")
+			(hide yes)
+			(effects
+				(font
+					(size 1 1)
+					(thickness 0.15)
+				)
+			)
+		)
+		(property "Value" "MountingHole"
+			(at 0 3.15 0)
+			(layer "F.Fab")
+			(hide yes)
+			(effects
+				(font
+					(size 1 1)
+					(thickness 0.15)
+				)
+			)
+		)
+		(property "Datasheet" "~"
+			(at 0 0 0)
+			(layer "F.Fab")
+			(hide yes)
+			(effects
+				(font
+					(size 1.27 1.27)
+					(thickness 0.15)
+				)
+			)
+		)
+		(property "Description" "Mounting Hole without connection"
+			(at 0 0 0)
+			(layer "F.Fab")
+			(hide yes)
+			(effects
+				(font
+					(size 1.27 1.27)
+					(thickness 0.15)
+				)
+			)
+		)
+		(property ki_fp_filters "MountingHole*")
+		(sheetname "/")
+		(sheetfile "mubi-bot-3.kicad_sch")
+		(attr exclude_from_pos_files exclude_from_bom)
+		(fp_circle
+			(center 0 0)
+			(end 2.2 0)
+			(stroke
+				(width 0.15)
+				(type solid)
+			)
+			(fill no)
+			(layer "Cmts.User")
+		)
+		(fp_circle
+			(center 0 0)
+			(end 2.45 0)
+			(stroke
+				(width 0.05)
+				(type solid)
+			)
+			(fill no)
+			(layer "F.CrtYd")
+		)
+		(fp_text user "${REFERENCE}"
+			(at 0 0 0)
+			(layer "F.Fab")
+			(effects
+				(font
+					(size 1 1)
+					(thickness 0.15)
+				)
+			)
+		)
+		(pad "" np_thru_hole circle
+			(at 0 0)
+			(size 2.2 2.2)
+			(drill 2.2)
+			(layers "*.Cu" "*.Mask")
+		)
 		(embedded_fonts no)
 	)
@@
 	)
 	(segment
+		(start 135.0136 95.4736)
+		(end 135.0136 91.028599)
+		(width 1.27)
+		(layer "B.Cu")
+		(net 1)
+	)
+	(segment
 		(start 172.4786 89.1236)
 		(end 172.4786 88.4886)
 		(width 1.016)
-		(layer "B.Cu")
-		(net 1)
-	)
-	(segment
-		(start 135.0136 91.0286)
-		(end 131.8386 87.8536)
-		(width 1.27)
 		(layer "B.Cu")
 		(net 1)
@@
 	)
 	(segment
+		(start 136.9186 97.3786)
+		(end 135.0136 95.4736)
+		(width 1.27)
+		(layer "B.Cu")
+		(net 1)
+	)
+	(segment
 		(start 143.2686 87.8536)
 		(end 146.4436 84.6786)
@@
 	)
 	(segment
-		(start 131.8386 87.8536)
-		(end 131.2036 87.8536)
-		(width 1.27)
-		(layer "B.Cu")
-		(net 1)
-	)
-	(segment
 		(start 144.5386 92.9336)
 		(end 143.2686 91.6636)
@@
 	)
 	(segment
+		(start 131.838601 87.8536)
+		(end 131.2036 87.8536)
+		(width 1.27)
+		(layer "B.Cu")
+		(net 1)
+	)
+	(segment
 		(start 159.7786 89.7586)
 		(end 158.5086 89.7586)
@@
 	)
 	(segment
-		(start 135.0136 95.4736)
-		(end 135.0136 91.0286)
+		(start 131.2036 87.8536)
+		(end 127.1142 87.8536)
+		(width 2.54)
+		(layer "B.Cu")
+		(net 1)
+	)
+	(segment
+		(start 160.4136 102.4586)
+		(end 161.0486 102.4586)
 		(width 1.27)
+		(layer "B.Cu")
+		(net 1)
+	)
+	(segment
+		(start 148.3486 114.5236)
+		(end 148.9836 113.8886)
+		(width 1.6764)
+		(layer "B.Cu")
+		(net 1)
+	)
+	(segment
+		(start 130.5686 87.2186)
+		(end 131.2036 87.8536)
+		(width 2.54)
+		(layer "B.Cu")
+		(net 1)
+	)
+	(segment
+		(start 148.3486 115.7936)
+		(end 148.3486 114.5236)
+		(width 1.6764)
 		(layer "B.Cu")
 		(net 1)
@@
 	)
 	(segment
-		(start 131.2036 87.8536)
-		(end 127.1142 87.8536)
-		(width 2.54)
-		(layer "B.Cu")
-		(net 1)
-	)
-	(segment
-		(start 160.4136 102.4586)
-		(end 161.0486 102.4586)
-		(width 1.27)
-		(layer "B.Cu")
-		(net 1)
-	)
-	(segment
-		(start 148.3486 114.5236)
-		(end 148.9836 113.8886)
-		(width 1.6764)
-		(layer "B.Cu")
-		(net 1)
-	)
-	(segment
-		(start 130.5686 87.2186)
-		(end 131.2036 87.8536)
-		(width 2.54)
-		(layer "B.Cu")
-		(net 1)
-	)
-	(segment
-		(start 148.3486 115.7936)
-		(end 148.3486 114.5236)
-		(width 1.6764)
-		(layer "B.Cu")
-		(net 1)
-	)
-	(segment
 		(start 154.0636 92.2986)
 		(end 155.9686 92.2986)
@@
 		(end 139.4586 97.3786)
 		(width 1.778)
+		(layer "B.Cu")
+		(net 1)
+	)
+	(segment
+		(start 135.0136 91.028599)
+		(end 131.838601 87.8536)
+		(width 1.27)
 		(layer "B.Cu")
 		(net 1)
@@
 	)
 	(segment
-		(start 136.9186 97.3786)
-		(end 135.0136 95.4736)
-		(width 1.27)
-		(layer "B.Cu")
-		(net 1)
-	)
-	(segment
 		(start 159.1436 102.4586)
 		(end 157.2386 102.4586)
@@
 	)
 	(segment
-		(start 135.6486 85.9486)
+		(start 143.9036 84.6786)
+		(end 141.3814 84.6786)
+		(width 0.6096)
+		(layer "F.Cu")
+		(net 4)
+	)
+	(segment
+		(start 135.6486 90.4114)
 		(end 135.6486 117.6986)
 		(width 0.6096)
@@
 	)
 	(segment
-		(start 143.9036 84.6786)
-		(end 136.9186 84.6786)
+		(start 141.3814 84.6786)
+		(end 135.6486 90.4114)
 		(width 0.6096)
 		(layer "F.Cu")
-		(net 4)
-	)
-	(segment
-		(start 136.9186 84.6786)
-		(end 135.6486 85.9486)
-		(width 0.6096)
-		(layer "F.Cu")

Commit message: update mubi-bot
Parts:
- added ARDUINO_NANO1: ARDUINO_NANO, mubi-bot-3:ARDUINO_NANO, F.Cu at (304.5, 133.3)
- added ARDUINO_NANO1: ARDUINO_NANO, mubi-bot-3:ARDUINO_NANO, F.Cu at (306.3, 64.7)
- added ARDUINO_NANO1: ARDUINO_NANO, mubi-bot-3:ARDUINO_NANO, F.Cu at (178.8, 64.5)
- added ARDUINO_NANO1: ARDUINO_NANO, mubi-bot-3:ARDUINO_NANO, F.Cu at (241.3, 133.3)
- added ARDUINO_NANO1: ARDUINO_NANO, mubi-bot-3:ARDUINO_NANO, F.Cu at (112.4, 64.5)
- added ARDUINO_NANO1: ARDUINO_NANO, mubi-bot-3:ARDUINO_NANO, F.Cu at (243.1, 64.7)
- added ARDUINO_NANO1: ARDUINO_NANO, mubi-bot-3:ARDUINO_NANO, F.Cu at (177.1, 133.2)
- added ARDUINO_NANO1: ARDUINO_NANO, mubi-bot-3:ARDUINO_NANO, F.Cu at (110.6, 133.1)
- added ARDUINO_NANO1: ARDUINO_NANO, mubi-bot-3:ARDUINO_NANO, F.Cu at (46.4, 133.0)
- added C1: C-EU050-025X075, mubi-bot-3:C050-025X075, F.Cu at (317.2, 121.3)
- added C1: C-EU050-025X075, mubi-bot-3:C050-025X075, F.Cu at (123.3, 121.1)
- added C1: C-EU050-025X075, mubi-bot-3:C050-025X075, F.Cu at (189.8, 121.2)
- added C1: C-EU050-025X075, mubi-bot-3:C050-025X075, F.Cu at (255.8, 52.6)
- added C1: C-EU050-025X075, mubi-bot-3:C050-025X075, F.Cu at (191.5, 52.5)
- added C1: C-EU050-025X075, mubi-bot-3:C050-025X075, F.Cu at (319.0, 52.6)
- added C1: C-EU050-025X075, mubi-bot-3:C050-025X075, F.Cu at (254.0, 121.3)
- added C1: C-EU050-025X075, mubi-bot-3:C050-025X075, F.Cu at (125.1, 52.4)
- added C1: C-EU050-025X075, mubi-bot-3:C050-025X075, F.Cu at (59.1, 121.0)
- added C2: CPOL-EUE2.5-5, mubi-bot-3:E2,5-5, F.Cu at (124.5, 43.5)
- added C2: CPOL-EUE2.5-5, mubi-bot-3:E2,5-5, F.Cu at (190.9, 43.6)
- added C2: CPOL-EUE2.5-5, mubi-bot-3:E2,5-5, F.Cu at (122.7, 112.2)
- added C2: CPOL-EUE2.5-5, mubi-bot-3:E2,5-5, F.Cu at (58.4, 112.1)
- added C2: CPOL-EUE2.5-5, mubi-bot-3:E2,5-5, F.Cu at (318.3, 43.7)
- added C2: CPOL-EUE2.5-5, mubi-bot-3:E2,5-5, F.Cu at (189.1, 112.3)
- added C2: CPOL-EUE2.5-5, mubi-bot-3:E2,5-5, F.Cu at (255.2, 43.7)
- added C2: CPOL-EUE2.5-5, mubi-bot-3:E2,5-5, F.Cu at (253.4, 112.4)
- added C2: CPOL-EUE2.5-5, mubi-bot-3:E2,5-5, F.Cu at (316.5, 112.4)
- added H1: MountingHole, MountingHole:MountingHole_2.2mm_M2, F.Cu at (294.4, 46.0)
- added H1: MountingHole, MountingHole:MountingHole_2.2mm_M2, F.Cu at (100.6, 45.8)
- added H1: MountingHole, MountingHole:MountingHole_2.2mm_M2, F.Cu at (231.3, 46.0)
- added H1: MountingHole, MountingHole:MountingHole_2.2mm_M2, F.Cu at (98.8, 114.5)
- added H1: MountingHole, MountingHole:MountingHole_2.2mm_M2, F.Cu at (34.5, 114.4)
- added H1: MountingHole, MountingHole:MountingHole_2.2mm_M2, F.Cu at (292.7, 114.7)
- added H1: MountingHole, MountingHole:MountingHole_2.2mm_M2, F.Cu at (167.0, 45.9)
- added H1: MountingHole, MountingHole:MountingHole_2.2mm_M2, F.Cu at (165.2, 114.6)
- added H1: MountingHole, MountingHole:MountingHole_2.2mm_M2, F.Cu at (229.5, 114.7)
- added H2: MountingHole, MountingHole:MountingHole_2.2mm_M2, F.Cu at (257.9, 82.8)
- added H2: MountingHole, MountingHole:MountingHole_2.2mm_M2, F.Cu at (319.3, 151.5)
- added H2: MountingHole, MountingHole:MountingHole_2.2mm_M2, F.Cu at (321.1, 82.8)
- added H2: MountingHole, MountingHole:MountingHole_2.2mm_M2, F.Cu at (191.9, 151.4)
- added H2: MountingHole, MountingHole:MountingHole_2.2mm_M2, F.Cu at (125.5, 151.3)
- added H2: MountingHole, MountingHole:MountingHole_2.2mm_M2, F.Cu at (193.7, 82.7)
- added H2: MountingHole, MountingHole:MountingHole_2.2mm_M2, F.Cu at (127.2, 82.6)
- added H2: MountingHole, MountingHole:MountingHole_2.2mm_M2, F.Cu at (61.2, 151.2)
- added H2: MountingHole, MountingHole:MountingHole_2.2mm_M2, F.Cu at (256.1, 151.5)
- added IC1: L293D, mubi-bot-3:DIL16, F.Cu at (178.8, 74.7)
- added IC1: L293D, mubi-bot-3:DIL16, F.Cu at (177.1, 143.4)
- added IC1: L293D, mubi-bot-3:DIL16, F.Cu at (306.3, 74.8)
- added IC1: L293D, mubi-bot-3:DIL16, F.Cu at (304.5, 143.5)
- added IC1: L293D, mubi-bot-3:DIL16, F.Cu at (112.4, 74.6)
- added IC1: L293D, mubi-bot-3:DIL16, F.Cu at (110.6, 143.3)
- added IC1: L293D, mubi-bot-3:DIL16, F.Cu at (243.1, 74.8)
- added IC1: L293D, mubi-bot-3:DIL16, F.Cu at (241.3, 143.5)
- added IC1: L293D, mubi-bot-3:DIL16, F.Cu at (46.4, 143.2)
- added J1: SEL, Connector_PinHeader_2.54mm:PinHeader_1x03_P2.54mm_Vertical, F.Cu at (105.1, 110.7)
- added J1: SEL, Connector_PinHeader_2.54mm:PinHeader_1x03_P2.54mm_Vertical, F.Cu at (40.9, 110.6)
- added J1: SEL, Connector_PinHeader_2.54mm:PinHeader_1x03_P2.54mm_Vertical, F.Cu at (300.8, 42.2)
- added J1: SEL, Connector_PinHeader_2.54mm:PinHeader_1x03_P2.54mm_Vertical, F.Cu at (106.9, 42.0)
- added J1: SEL, Connector_PinHeader_2.54mm:PinHeader_1x03_P2.54mm_Vertical, F.Cu at (173.4, 42.1)
- added J1: SEL, Connector_PinHeader_2.54mm:PinHeader_1x03_P2.54mm_Vertical, F.Cu at (171.6, 110.8)
- added J1: SEL, Connector_PinHeader_2.54mm:PinHeader_1x03_P2.54mm_Vertical, F.Cu at (235.8, 110.9)
- added J1: SEL, Connector_PinHeader_2.54mm:PinHeader_1x03_P2.54mm_Vertical, F.Cu at (237.6, 42.2)
- added J1: SEL, Connector_PinHeader_2.54mm:PinHeader_1x03_P2.54mm_Vertical, F.Cu at (299.0, 110.9)
- added PAD1: WIREPAD1,6/0,9, mubi-bot-3:1,6_0,9, F.Cu at (106.2, 154.1)
- added PAD1: WIREPAD1,6/0,9, mubi-bot-3:1,6_0,9, F.Cu at (172.6, 154.2)
- added PAD1: WIREPAD1,6/0,9, mubi-bot-3:1,6_0,9, F.Cu at (300.0, 154.3)
- added PAD1: WIREPAD1,6/0,9, mubi-bot-3:1,6_0,9, F.Cu at (238.6, 85.6)
- added PAD1: WIREPAD1,6/0,9, mubi-bot-3:1,6_0,9, F.Cu at (41.9, 154.0)
- added PAD1: WIREPAD1,6/0,9, mubi-bot-3:1,6_0,9, F.Cu at (174.4, 85.5)
- added PAD1: WIREPAD1,6/0,9, mubi-bot-3:1,6_0,9, F.Cu at (108.0, 85.4)
- added PAD1: WIREPAD1,6/0,9, mubi-bot-3:1,6_0,9, F.Cu at (301.8, 85.6)
- added PAD1: WIREPAD1,6/0,9, mubi-bot-3:1,6_0,9, F.Cu at (236.9, 154.3)
- added PAD2: WIREPAD1,6/0,9, mubi-bot-3:1,6_0,9, F.Cu at (300.7, 127.0)
- added PAD2: WIREPAD1,6/0,9, mubi-bot-3:1,6_0,9, F.Cu at (106.8, 126.8)
- added PAD2: WIREPAD1,6/0,9, mubi-bot-3:1,6_0,9, F.Cu at (175.0, 58.2)
- added PAD2: WIREPAD1,6/0,9, mubi-bot-3:1,6_0,9, F.Cu at (302.5, 58.3)
- added PAD2: WIREPAD1,6/0,9, mubi-bot-3:1,6_0,9, F.Cu at (239.3, 58.3)
- added PAD2: WIREPAD1,6/0,9, mubi-bot-3:1,6_0,9, F.Cu at (42.5, 126.7)
- added PAD2: WIREPAD1,6/0,9, mubi-bot-3:1,6_0,9, F.Cu at (173.2, 126.9)
- added PAD2: WIREPAD1,6/0,9, mubi-bot-3:1,6_0,9, F.Cu at (237.5, 127.0)
- added PAD2: WIREPAD1,6/0,9, mubi-bot-3:1,6_0,9, F.Cu at (108.6, 58.1)
- added SV1: MA05-1, mubi-bot-3:MA05-1, F.Cu at (319.0, 64.7)
- added SV1: MA05-1, mubi-bot-3:MA05-1, F.Cu at (125.1, 64.5)
- added SV1: MA05-1, mubi-bot-3:MA05-1, F.Cu at (254.0, 133.3)
- added SV1: MA05-1, mubi-bot-3:MA05-1, F.Cu at (189.8, 133.2)
- added SV1: MA05-1, mubi-bot-3:MA05-1, F.Cu at (59.1, 133.0)
- added SV1: MA05-1, mubi-bot-3:MA05-1, F.Cu at (191.5, 64.5)
- added SV1: MA05-1, mubi-bot-3:MA05-1, F.Cu at (317.2, 133.3)
- added SV1: MA05-1, mubi-bot-3:MA05-1, F.Cu at (123.3, 133.1)
- added SV1: MA05-1, mubi-bot-3:MA05-1, F.Cu at (255.8, 64.7)
- added X1: AK500/10-H, mubi-bot-3:AK500_10-H, F.Cu at (159.2, 64.5)
- added X1: AK500/10-H, mubi-bot-3:AK500_10-H, F.Cu at (90.9, 133.1)
- added X1: AK500/10-H, mubi-bot-3:AK500_10-H, F.Cu at (286.6, 64.7)
- added X1: AK500/10-H, mubi-bot-3:AK500_10-H, F.Cu at (26.7, 133.0)
- added X1: AK500/10-H, mubi-bot-3:AK500_10-H, F.Cu at (221.6, 133.3)
- added X1: AK500/10-H, mubi-bot-3:AK500_10-H, F.Cu at (92.7, 64.5)
- added X1: AK500/10-H, mubi-bot-3:AK500_10-H, F.Cu at (223.4, 64.7)
- added X1: AK500/10-H, mubi-bot-3:AK500_10-H, F.Cu at (284.8, 133.3)
- added X1: AK500/10-H, mubi-bot-3:AK500_10-H, F.Cu at (157.4, 133.2)
- added X2: AK500/10-H, mubi-bot-3:AK500_10-H, F.Cu at (201.1, 64.5)
- added X2: AK500/10-H, mubi-bot-3:AK500_10-H, F.Cu at (263.5, 133.3)
- added X2: AK500/10-H, mubi-bot-3:AK500_10-H, F.Cu at (265.3, 64.7)
- added X2: AK500/10-H, mubi-bot-3:AK500_10-H, F.Cu at (132.8, 133.1)
- added X2: AK500/10-H, mubi-bot-3:AK500_10-H, F.Cu at (326.7, 133.3)
- added X2: AK500/10-H, mubi-bot-3:AK500_10-H, F.Cu at (199.3, 133.2)
- added X2: AK500/10-H, mubi-bot-3:AK500_10-H, F.Cu at (134.6, 64.5)
- added X2: AK500/10-H, mubi-bot-3:AK500_10-H, F.Cu at (68.6, 133.0)
- added X2: AK500/10-H, mubi-bot-3:AK500_10-H, F.Cu at (328.5, 64.7)
- moved PAD1 106.4 mm to (43.7, 85.3)
- moved ARDUINO_NANO1 106.4 mm to (48.1, 64.3)
- moved C1 106.4 mm to (60.8, 52.3)
- moved C2 106.4 mm to (60.2, 43.4)
- moved H1 106.4 mm to (36.3, 45.7)
- moved H2 106.4 mm to (63.0, 82.5)
- moved IC1 106.4 mm to (48.1, 74.5)
- moved J1 106.4 mm to (42.7, 41.9)
- moved PAD2 106.4 mm to (44.3, 58.0)
- moved SV1 106.4 mm to (60.8, 64.3)
- moved X1 106.4 mm to (28.5, 64.3)
- moved X2 106.4 mm to (70.4, 64.3)
Routing:
- net GND: track 191.1 -> 1911.2 mm, vias 4 -> 40
- net +5V: track 109.3 -> 1093.1 mm
- net /+VBAT: track 77.3 -> 773.4 mm, vias 3 -> 30
- net /M1B: track 52.0 -> 520.1 mm
- net /M2B: track 45.1 -> 451.4 mm
- net Net-(ARDUINO_NANO1-D9/OC1A): track 44.7 -> 446.5 mm, vias 2 -> 20
- net /M1A: track 40.8 -> 407.7 mm
- net /M2A: track 40.5 -> 404.8 mm
- net /ENA1: track 33.2 -> 332.2 mm, vias 2 -> 20
- net /AUX2: track 22.3 -> 223.2 mm
- net /SCL: track 22.0 -> 219.8 mm
- net /TRIG: track 21.2 -> 212.2 mm
- net /ECHO3: track 19.3 -> 192.7 mm
- net /SDA: track 18.6 -> 186.4 mm
- net /ECHO2: track 18.2 -> 182.5 mm
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Other:
- board size 49.8 x 50.8 mm -> 309.8 x 119.8 mm
